File: PCB_Design/WalkmanPCB_V1/WalkmanPCB_V1.kicad_sch (KiCad schematic)
At the start: 41 parts, among them U1 VS1053B, U2 ESP32-S3-WROOM-1, Y1 12.288 MHz

Commit message: Updated schematics with a headphone amp. WIP
Parts:
- added C21, C23, C24, C25, C26, C27, C28, C29, C30, C33, C40, C41, C43, C45: 0.1uF, Capacitor_SMD:C_0603_1608Metric, symbol Device:C_Small
- added C22, C31, C34, C35, C36, C37, C38, C39, C42, C44, C46: 10uF, Capacitor_SMD:C_0603_1608Metric, symbol Device:C_Small
- added C32, C47, C48, C49: 1uF, Capacitor_SMD:C_0603_1608Metric, symbol Device:C_Small
- added D1, D2: LED, symbol Device:LED
- added FB1, FB2, FB3: 120E, Resistor_SMD:R_0603_1608Metric, symbol Device:FerriteBead_Small
- added H1, H2, H3, H4: MountingHole, MountingHole:MountingHole_3.2mm_M3, symbol Mechanical:MountingHole
- added J1: Conn_01x04_Pin, Connector_PinHeader_2.54mm:PinHeader_1x04_P2.54mm_Vertical, symbol Connector:Conn_01x04_Pin
- added J2: Micro_SD_Card_Det1, Connector_Card:microSD_HC_Hirose_DM3AT-SF-PEJM5, symbol Connector:Micro_SD_Card_Det1
- added J3: SJ1-3545N, GlobalFP:CUI_SJ1-3545N, symbol SJ1-3545N:SJ1-3545N
- added J4: USB_C_Receptacle_USB2.0_16P, Connector_USB:USB_C_Receptacle_XKB_U262-16XN-4BVC11, symbol Connector:USB_C_Receptacle_USB2.0_16P
- added J5: Conn_01x02_Pin, Connector_JST:JST_EH_B2B-EH-A_1x02_P2.50mm_Vertical, symbol Connector:Conn_01x02_Pin
- added R19, R20: 0E, Resistor_SMD:R_0603_1608Metric, symbol Device:R_Small
- added R21, R22, R23, R24, R25, R26, R27, R28: 10K, Resistor_SMD:R_0603_1608Metric, symbol Device:R_Small
- added R29, R30: 0E, symbol Device:R
- added R31, R32: 5.1K, Resistor_SMD:R_0603_1608Metric, symbol Device:R_Small
- added R33: 1.2K, Resistor_SMD:R_0603_1608Metric, symbol Device:R_Small
- added R34, R35: 1K, Resistor_SMD:R_0603_1608Metric, symbol Device:R_Small
- added SW1, SW2: SW_Push, symbol Switch:SW_Push
- added SW3, SW4, SW5, SW6, SW7: SW_Push, Button_Switch_THT:SW_PUSH-12mm, symbol Switch:SW_Push
- added SW8: SW_SPDT, symbol Switch:SW_SPDT
- added U3: USBLC6-2SC6, Package_TO_SOT_SMD:SOT-23-6, symbol Power_Protection:USBLC6-2SC6
- added U4: TP4056-42-ESOP8, Package_SO:SOIC-8-1EP_3.9x4.9mm_P1.27mm_EP2.41x3.3mm_ThermalVias, symbol Battery_Management:TP4056-42-ESOP8
- added U5: XC6220B331MR, Package_TO_SOT_SMD:SOT-23-5, symbol Regulator_Linear:XC6220B331MR
- added U6: AP2112K-1.8, Package_TO_SOT_SMD:SOT-23-5, symbol Regulator_Linear:AP2112K-1.8
- added U7: MAX97220DETE_, MAX97220DETE_:QFN50P300X300X80-17N, symbol MAX97220DETE_:MAX97220DETE_
- C1, C10, C11, C12, C13, C14, C15, C16, C17, C18, C19, C2, C20, C3, C4, C5, C6, C7, C8, C9: footprint (none) -> Capacitor_SMD:C_0603_1608Metric
- R1, R10, R11, R12, R13, R14, R15, R16, R17, R18, R2, R3, R4, R5, R6, R7, R8, R9: footprint (none) -> Resistor_SMD:R_0603_1608Metric
- U1: footprint Adafruit VS1053 Breakout:LQFP48 -> Package_QFP:LQFP-48_7x7mm_P0.5mm
- Y1: footprint (none) -> Crystal:Crystal_SMD_HC49-SD_HandSoldering
Connections:
- net +1V8: now also C45.1, C46.1, U6.5 (VOUT)
- net +3V3: now also U2.2 (3V3), C21.2, C22.2, C30.2, C31.2, C32.2, C33.2, C34.2, C41.1, C42.1, C43.1, C44.1, FB2.1, J1.1 (Pin_1), J2.4 (VDD), R21.2, R22.2, R23.2, R24.2, R25.2, R26.2, R27.2, R28.2, U5.5 (VOUT), U6.1 (VIN), U6.3 (EN)
- net GND: now also U2.1 (GND), U2.40 (GND), U2.41 (GND), C21.1, C22.1, C23.1, C24.1, C25.1, C26.1, C27.1, C28.1, C29.1, C30.1, C31.1, C32.1, C33.1, C34.1, C35.2, C36.2, C37.2, C38.2, C39.2, C40.2, C41.2, C42.2, C43.2, C44.2, C45.2, C46.2, FB3.1, J1.4 (Pin_4), J2.10 (SHIELD), J2.6 (VSS), J4.A1 (GND), J4.A12 (GND), J4.B1 (GND), J4.B12 (GND), J4.S1 (SHIELD), J5.1 (Pin_1), R31.2, R32.2, R33.1, SW1.1, SW2.1, SW3.1, SW4.1, SW5.1, SW6.1, SW7.1, U3.2 (GND), U4.1 (TEMP), U4.3 (GND), U4.9 (EPAD), U5.2 (GND), U6.2 (GND)
- net GNDA: now also C47.1, C48.1, FB3.2
- net LEFT: now also R19.2
- net MISO: now also U2.21 (IO13), J2.7 (DAT0)
- net MOSI: now also U2.19 (IO11), J2.3 (CMD)
- net RIGHT: now also R20.2
- net SCLK: now also U2.20 (IO12), J2.5 (CLK)
- net VDDA: now also FB2.2
- net VS_RST: now also U2.22 (IO14)
- net at U2.13 (USB_D-): now also R29.1
- net at U2.14 (USB_D+): now also R30.1
- net SD_CS: now reaches U2.18 (IO10)
- net SD_CS: now also J2.2 (DAT3/CD), R21.1
- net BOOT: now reaches U2.27 (IO0)
- net BOOT: now also C24.2, R23.1, SW2.2
- net EN: now reaches U2.3 (EN)
- net EN: now also C23.2, R22.1, SW1.2
- new net: D2.1 (K), U4.7 (~{CHRG})
- new net: D2.2 (A), R35.2
- new net: C49.1, U7.2 (C1P)
- new net: C49.2, U7.4 (C1N)
- new net: D1.1 (K), U4.6 (~{STDBY})
- new net: D1.2 (A), R34.2
- new net: J4.B5 (CC2), R32.1
- new net: R33.2, U4.2 (PROG)
- new net: J4.A5 (CC1), R31.1
- new net Button1: C25.2, R24.1, SW3.2
- new net Button2: C26.2, R25.1, SW4.2
- new net Button3: C27.2, R26.1, SW5.2
- new net Button4: C28.2, R27.1, SW6.2
- new net Button5: C29.2, R28.1, SW7.2
- new net Card_Det: J2.9 (DET)
- new net D+: J4.A6 (D+), J4.B6 (D+), R30.2, U3.3 (I/O2), U3.4 (I/O2)
- new net D-: J4.A7 (D-), J4.B7 (D-), R29.2, U3.1 (I/O1), U3.6 (I/O1)
- new net Disp_SCL: J1.2 (Pin_2)
- new net Disp_SDA: J1.3 (Pin_3)
- new net GBUFJ: J3.1
- new net LEFTA: R19.1
- new net LEFTJ: J3.2
- new net RIGHTA: R20.1
- new net RIGHTJ: J3.3
- new net VBAT_CHG: C37.1, J5.2 (Pin_2), SW8.1 (A), U4.5 (BAT)
- new net VBAT_SYS: C39.1, C40.1, C47.2, C48.2, SW8.2 (B), U5.1 (VIN), U5.3 (CE), U7.1 (PVDD), U7.13 (SVDD)
- new net VBUS: C35.1, FB1.1, J4.A4 (VBUS), J4.A9 (VBUS), J4.B4 (VBUS), J4.B9 (VBUS), U3.5 (VBUS)
- new net VBUSF: C36.1, C38.1, FB1.2, R34.1, R35.1, U4.4 (V_{CC}), U4.8 (CE)
- no-connect marks 2 -> 9
Other:
- note added: "Battery Connector"
- note added: "DM3AT-SF-PEJM5(41)"
- note added: "Display"
- note added: "Headphone Jack + Headphone Amplifier"
- note added: "SD Card"

Commit message: Refactored power manager, changed headphone amp to PAM8908 in shcematics.
Parts:
- removed C47: 1uF, Capacitor_SMD:C_0603_1608Metric, symbol Device:C_Small
- removed U7: MAX97220DETE_, MAX97220DETE_:QFN50P300X300X80-17N, symbol MAX97220DETE_:MAX97220DETE_
- added C50, C51, C53, C54, C55, C56: 1uF, Capacitor_SMD:C_0603_1608Metric, symbol Device:C_Small
- added C52: 2.2uF, Capacitor_SMD:C_0603_1608Metric, symbol Device:C_Small
- added FB4: 120E, Resistor_SMD:R_0603_1608Metric, symbol Device:FerriteBead_Small
- added R36, R37, R38: 10K, Resistor_SMD:R_0603_1608Metric, symbol Device:R_Small
- added SW9: RotaryEncoder_Switch, symbol Device:RotaryEncoder_Switch
- added U8: PAM8908, Package_DFN_QFN:QFN-16-1EP_3x3mm_P0.5mm_EP1.7x1.7mm, symbol Amplifier_Audio:PAM8908
- C48: value 1uF -> 10uF
- D1, D2: footprint (none) -> LED_SMD:LED_0603_1608Metric
- R29, R30: footprint (none) -> Resistor_SMD:R_0603_1608Metric
Connections:
- net GBUFJ is gone; now on net GND: J3.1
- net +3V3: now also R36.2, R37.2
- net GND: now also C48.1, C49.1, C51.1, C52.1, C55.2, C56.2, FB4.2, R38.2
- net GNDA: no longer C48.1
- net LEFTA: now also C53.2
- net RIGHTA: now also C54.2
- net VBAT_SYS: now also C52.2, U8.14 (PVDD)
- net at C49.2: now also U8.8 (HPVSS)
- net LEFTJ renamed RIGHT_OUT
- net RIGHT_OUT: now also U8.5 (OUTR)
- net RIGHTJ renamed LEFT_OUT
- net LEFT_OUT: now also U8.16 (OUTL)
- new net: C53.1, U8.1 (INL-)
- new net: C56.1, U8.3 (INR+)
- new net: C54.1, U8.4 (INR-)
- new net: C51.2, U8.12 (HPVDD)
- new net: C50.2, U8.11 (CAP+)
- new net: C55.1, U8.2 (INL+)
- new net: R37.1, U8.6 (G0)
- new net: R38.1, U8.7 (G1)
- new net: C50.1, U8.9 (CAP-)
- new net AUDIO_GND: FB4.1, U8.10 (PGND), U8.15 (SGND), U8.17 (EPAD)
- new net EN_AMP: R36.1, U8.13 (EN)
- no-connect marks 9 -> 11

Commit message: Minor Updates to the Schematics, removed headphone Amp IC
Parts:
- removed C51, C53, C54, C55, C56: 1uF, Capacitor_SMD:C_0603_1608Metric, symbol Device:C_Small
- removed C52: 2.2uF, Capacitor_SMD:C_0603_1608Metric, symbol Device:C_Small
- removed FB3, FB4: 120E, Resistor_SMD:R_0603_1608Metric, symbol Device:FerriteBead_Small
- removed U8: PAM8908, Package_DFN_QFN:QFN-16-1EP_3x3mm_P0.5mm_EP1.7x1.7mm, symbol Amplifier_Audio:PAM8908
- added C47: 470uF, symbol Device:C_Polarized_Small
- added R39, R40: 10K, Resistor_SMD:R_0603_1608Metric, symbol Device:R_Small
- C48: value 10uF -> 0.1uF
- C49, C50: value 1uF -> 0.1uF
- R36, R37: value 10K -> 0E
Connections:
- net EN_AMP is gone; now on net GND: R36.1
- net +3V3: now also R38.2, C47.1, R39.2, R40.2; no longer R1.1, R36.2, R37.2
- net Button1: now also U2.5 (IO5)
- net Button2: now also U2.6 (IO6)
- net Button3: now also U2.7 (IO7)
- net Button4: now also U2.12 (IO8)
- net DREQ: now also U2.8 (IO15)
- net GBUF: now also R37.2
- net GND: now also C50.1, SW9.C, SW9.S2, C47.2; no longer J3.1, R38.2
- net GNDA: now also R36.2
- net VBAT_SYS: no longer C48.2
- net VDDA: now also R1.1
- net XDCS: now also U2.9 (IO16)
- net R_S: now reaches C50.2
- net R_S: now also SW9.S1, R40.1
- net GBUFA: now reaches R37.1
- net GBUFA: now also J3.1
- net Rotary1: now reaches R38.1
- net Rotary1: now also C48.2, SW9.A
- net Rotary2: now reaches C49.2
- net Rotary2: now also SW9.B, R39.1
- no-connect marks 11 -> 12
Other:
- note added: "DC Blocking//DNP"
- note added: "DNP//STAR"
- note added: "Dreq"
- note added: "JACK"
- note added: "Xdcs"
- note removed: "Headphone Jack + Headphone Amplifier"
- moved on the sheet: C18, C19, C20, J3, R16, R17, R18, R19, R20, SW9

Commit message: Updated Routing for PCB
Parts:
- removed C29: 0.1uF, Capacitor_SMD:C_0603_1608Metric, symbol Device:C_Small
- removed R28: 10K, Resistor_SMD:R_0603_1608Metric, symbol Device:R_Small
- removed R36: 0E, Resistor_SMD:R_0603_1608Metric, symbol Device:R_Small
- removed SW7: SW_Push, Button_Switch_THT:SW_PUSH-12mm, symbol Switch:SW_Push
- removed Y1: 12.288 MHz, Crystal:Crystal_SMD_HC49-SD_HandSoldering, symbol Device:Crystal
- added R28, R41: 10K, Resistor_SMD:R_0603_1608Metric, symbol Device:R
- added Y1: AB308-12.288MHZ, GlobalFP:XTAL_AB308-12.288MHZ, symbol AB308-12.288MHZ:AB308-12.288MHZ
- C47: footprint (none) -> Capacitor_THT:C_Axial_L5.1mm_D3.1mm_P12.50mm_Horizontal
- C48, C49: value 0.1uF -> 10nF
- R33: value 1.2K -> 2K
- SW1, SW2: footprint (none) -> Button_Switch_THT:SW_Tactile_SPST_Angled_PTS645Vx58-2LFS
- SW3, SW4, SW5, SW6: footprint Button_Switch_THT:SW_PUSH-12mm -> Button_Switch_THT:SW_Tactile_SPST_Angled_PTS645Vx58-2LFS
- SW8: footprint (none) -> Button_Switch_THT:SW_Slide_SPDT_Angled_CK_OS102011MA1Q
- SW9: footprint (none) -> Rotary_Encoder:RotaryEncoder_Alps_EC11E-Switch_Vertical_H20mm
Connections:
- net GNDA is gone; now on net GND: C14.1, C15.1, C16.1, C17.1, C18.1, C19.1, C20.1, C4.2, R14.2, R15.2, U1.37 (AGND@0), U1.40 (AGND@1), U1.41 (AGND@2), U1.47 (AGND@3)
- net LEFT_OUT is gone; now on net RIGHTA: J3.3
- net RIGHT_OUT is gone; now on net LEFTA: J3.2
- net +3V3: now also R28.2, R41.2
- net Button4: now also U2.8 (IO15); no longer U2.12 (IO8)
- net Card_Det: now also U2.17 (IO9)
- net D+: no longer R30.2, U3.4 (I/O2)
- net D-: no longer R29.2, U3.6 (I/O1)
- net DREQ: now also U2.9 (IO16); no longer U2.8 (IO15)
- net Disp_SCL: now also J1.3 (Pin_3), U2.33 (IO40), R28.1; no longer J1.2 (Pin_2)
- net Disp_SDA: now also J1.4 (Pin_4), U2.34 (IO41), R41.1; no longer J1.3 (Pin_3)
- net GND: now also J1.2 (Pin_2); no longer J1.4 (Pin_4)
- net R_S: now also U2.4 (IO4)
- net Rotary1: now also U2.15 (IO3)
- net Rotary2: now also U2.12 (IO8)
- net XCS: now also U2.35 (IO42)
- net XDCS: now also U2.23 (IO21); no longer U2.9 (IO16)
- net DX-: now reaches R29.1, U2.13 (USB_D-)
- net at C2.1, R3.1, U1.17 (XTALOUT): now also Y1.1
- net at C3.1, R3.2, U1.18 (XTALIN): now also Y1.2
- net DX+: now reaches R30.1, U2.14 (USB_D+)
- new net DOUT+: R30.2, U3.4 (I/O2)
- new net DOUT-: R29.2, U3.6 (I/O1)
- no-connect marks 12 -> 25
Other:
- note added: "DC Blocking//DNP//Not Needed"
- note removed: "DC Blocking//DNP"
- note removed: "DNP//STAR"
- moved on the sheet: C48, C49, C50, R29, R30, R38, R39, R40, SW9
