File: PCB_Design/WalkmanPCB_V1/WalkmanPCB_V1.kicad_pcb (KiCad board)
At the start: 4 copper layers, 55 x 65 mm, 105 parts, among them J1 Conn_01x04_Pin, J2 Micro_SD_Card_Det1, J3 SJ1-3545N, J4 USB_C_Receptacle_USB2.0_16P, J5 Conn_01x02_Pin, SW3 SW_Push, SW4 SW_Push, SW5 SW_Push, SW6 SW_Push, SW7 SW_Push, U1 VS1053B, U2 ESP32-S3-WROOM-1, U3 USBLC6-2SC6, U4 TP4056-42-ESOP8, U5 XC6220B331MR, U6 AP2112K-1.8, Y1 12.288 MHz

Commit message: Refactored power manager, changed headphone amp to PAM8908 in shcematics.
Parts:
- removed the C30 at (155.1, 117.4)
- removed the C30 at (134.9, 99.4)
- removed the C34 at (134.9, 101.9)
- removed the C34 at (155.1, 120.0)
- added C30: 0.1uF, Capacitor_SMD:C_0603_1608Metric, F.Cu at (376.6, 215.5)
- added C34: 10uF, Capacitor_SMD:C_0603_1608Metric, F.Cu at (376.6, 225.5)
- added C48: 10uF, Capacitor_SMD:C_0603_1608Metric, F.Cu at (380.6, 223.0)
- added C49: 1uF, Capacitor_SMD:C_0603_1608Metric, F.Cu at (380.6, 225.5)
- added C50: 1uF, Capacitor_SMD:C_0603_1608Metric, F.Cu at (380.6, 228.0)
- added C51: 1uF, Capacitor_SMD:C_0603_1608Metric, F.Cu at (380.6, 230.5)
- added C52: 2.2uF, Capacitor_SMD:C_0603_1608Metric, F.Cu at (380.6, 233.1)
- added C53: 1uF, Capacitor_SMD:C_0603_1608Metric, F.Cu at (380.6, 235.6)
- added C54: 1uF, Capacitor_SMD:C_0603_1608Metric, F.Cu at (380.6, 238.1)
- added C55: 1uF, Capacitor_SMD:C_0603_1608Metric, F.Cu at (380.6, 240.6)
- added C56: 1uF, Capacitor_SMD:C_0603_1608Metric, F.Cu at (380.6, 243.1)
- added D1: LED, LED_SMD:LED_0603_1608Metric, F.Cu at (417.6, 206.9)
- added D2: LED, LED_SMD:LED_0603_1608Metric, F.Cu at (417.6, 209.5)
- added FB4: 120E, Resistor_SMD:R_0603_1608Metric, F.Cu at (384.6, 218.0)
- added R29: 0E, Resistor_SMD:R_0603_1608Metric, F.Cu at (392.6, 220.5)
- added R30: 0E, Resistor_SMD:R_0603_1608Metric, F.Cu at (392.6, 223.0)
- added R36: 10K, Resistor_SMD:R_0603_1608Metric, F.Cu at (392.6, 238.1)
- added R37: 10K, Resistor_SMD:R_0603_1608Metric, F.Cu at (392.6, 240.6)
- added R38: 10K, Resistor_SMD:R_0603_1608Metric, F.Cu at (392.6, 243.1)
- added U8: PAM8908, Package_DFN_QFN:QFN-16-1EP_3x3mm_P0.5mm_EP1.7x1.7mm, F.Cu at (426.6, 244.6)
- C18, C19, J2, J3, J4, R16, R17, R19, R20, U1, U2, Y1: moved to F.Cu
- moved H4 391.0 mm to (398.6, 239.5)
- moved U4 335.9 mm to (428.1, 238.7)
- moved U1 330.3 mm to (425.0, 227.4), turned to 0 degrees
- moved R20 321.1 mm to (388.6, 233.1), turned to 0 degrees
- moved J3 317.3 mm to (423.0, 184.9), turned to 0 degrees
- moved R17 315.0 mm to (388.6, 225.5), turned to 0 degrees
- moved Y1 314.1 mm to (413.2, 238.7)
- moved J1 313.3 mm to (423.0, 194.1), turned to 0 degrees
- moved H1 312.9 mm to (398.6, 215.7)
- moved U3 307.3 mm to (418.2, 194.2)
- moved U5 307.3 mm to (418.2, 198.8)
- moved U6 307.3 mm to (418.2, 203.4)
- moved R19 302.6 mm to (388.6, 230.5), turned to 0 degrees
- moved J4 301.3 mm to (425.1, 217.0), turned to 0 degrees
- moved C19 299.5 mm to (372.5, 223.0), turned to 0 degrees
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Connections:
- J3 pad 1: /GBUF -> GND
- J3 pad 2: /LEFTJ -> /RIGHT_OUT
- J3 pad 3: /RIGHTJ -> /LEFT_OUT
- R19 pad 1: /LEFTJ -> /LEFTA
- R20 pad 1: /RIGHTJ -> /RIGHTA
Routing:
- net /SCLK: vias 2 -> 0
- net /MOSI: vias 2 -> 0
- net /MISO: vias 2 -> 0
Other:
- board outline removed

Commit message: Basic 3D design of the case, updated pcb dimensions.
Parts:
- removed C1, C10, C11, C12, C13, C15, C16, C17, C21, C23, C24, C25, C26, C27, C28, C29, C30, C33, C40, C41, C43, C45, C6, C7, C8: 0.1uF, Capacitor_SMD:C_0603_1608Metric
- removed C14, C22, C31, C34, C35, C36, C37, C38, C39, C42, C44, C46, C48, C5, C9: 10uF, Capacitor_SMD:C_0603_1608Metric
- removed C18, C19: 10nF, Capacitor_SMD:C_0603_1608Metric
- removed C2, C3: 33pF, Capacitor_SMD:C_0603_1608Metric
- removed C20: 47nF, Capacitor_SMD:C_0603_1608Metric
- removed C32, C4, C49, C50, C51, C53, C54, C55, C56: 1uF, Capacitor_SMD:C_0603_1608Metric
- removed C52: 2.2uF, Capacitor_SMD:C_0603_1608Metric
- removed D1, D2: LED, LED_SMD:LED_0603_1608Metric
- removed FB1, FB2, FB3, FB4: 120E, Resistor_SMD:R_0603_1608Metric
- removed J1: Conn_01x04_Pin, Connector_PinHeader_2.54mm:PinHeader_1x04_P2.54mm_Vertical
- removed J5: Conn_01x02_Pin, Connector_JST:JST_EH_B2B-EH-A_1x02_P2.50mm_Vertical
- removed R1, R10, R11, R12, R13, R2, R4, R5, R6, R7, R8, R9: 100K, Resistor_SMD:R_0603_1608Metric
- removed R14, R15, R19, R20, R29, R30: 0E, Resistor_SMD:R_0603_1608Metric
- removed R16, R17: 20E, Resistor_SMD:R_0603_1608Metric
- removed R18: 10E, Resistor_SMD:R_0603_1608Metric
- removed R21, R22, R23, R24, R25, R26, R27, R28, R36, R37, R38: 10K, Resistor_SMD:R_0603_1608Metric
- removed R3: 1M, Resistor_SMD:R_0603_1608Metric
- removed R31, R32: 5.1K, Resistor_SMD:R_0603_1608Metric
- removed R33: 1.2K, Resistor_SMD:R_0603_1608Metric
- removed R34, R35: 1K, Resistor_SMD:R_0603_1608Metric
- removed SW3, SW4, SW5, SW6, SW7: SW_Push, Button_Switch_THT:SW_PUSH-12mm
- removed U3: USBLC6-2SC6, Package_TO_SOT_SMD:SOT-23-6
- removed U5: XC6220B331MR, Package_TO_SOT_SMD:SOT-23-5
- removed U6: AP2112K-1.8, Package_TO_SOT_SMD:SOT-23-5
- removed Y1: 12.288 MHz, Crystal:Crystal_SMD_HC49-SD_HandSoldering
- J2, J3, J4, U1, U2, U4, U8: moved to B.Cu
- moved U8 353.4 mm to (127.4, 56.4), turned to 180 degrees
- moved H1 347.4 mm to (95.8, 45.4)
- moved J3 345.9 mm to (107.3, 43.5), turned to -90 degrees
- moved U4 341.6 mm to (111.8, 109.8), turned to 180 degrees
- moved U1 332.4 mm to (135.8, 63.4), turned to 180 degrees
- moved J4 327.0 mm to (112.4, 121.6), turned to 180 degrees
- moved H3 322.5 mm to (95.8, 120.4)
- moved U2 314.1 mm to (103.6, 71.1), turned to -90 degrees
- moved H2 305.2 mm to (150.8, 45.4)
- moved J2 292.5 mm to (137.6, 116.8), turned to 180 degrees
- moved H4 274.9 mm to (150.8, 120.4)
Routing:
- removed copper zone on In1.Cu, net GND
- removed copper zone on In2.Cu, net GND
Other:
- board outline added: 65 x 85 mm

Commit message: Updated Routing for PCB
Parts:
- removed U8: PAM8908, Package_DFN_QFN:QFN-16-1EP_3x3mm_P0.5mm_EP1.7x1.7mm
- added C1: 0.1uF, Capacitor_SMD:C_0603_1608Metric, F.Cu at (154.1, 94.8)
- added C10: 0.1uF, Capacitor_SMD:C_0603_1608Metric, F.Cu at (150.0, 92.0)
- added C11: 0.1uF, Capacitor_SMD:C_0603_1608Metric, B.Cu at (140.8, 92.2)
- added C12: 0.1uF, Capacitor_SMD:C_0603_1608Metric, B.Cu at (146.0, 93.6)
- added C13: 0.1uF, Capacitor_SMD:C_0603_1608Metric, B.Cu at (140.6, 88.8)
- added C14: 10uF, Capacitor_SMD:C_0603_1608Metric, B.Cu at (145.6, 95.9)
- added C15: 0.1uF, Capacitor_SMD:C_0603_1608Metric, B.Cu at (140.2, 95.2)
- added C16: 0.1uF, Capacitor_SMD:C_0603_1608Metric, B.Cu at (147.2, 95.9)
- added C17: 0.1uF, Capacitor_SMD:C_0603_1608Metric, B.Cu at (141.9, 95.2)
- added C18: 10nF, Capacitor_SMD:C_0603_1608Metric, F.Cu at (144.0, 102.3)
- added C19: 10nF, Capacitor_SMD:C_0603_1608Metric, F.Cu at (140.8, 102.3)
- added C2: 33pF, Capacitor_SMD:C_0603_1608Metric, F.Cu at (144.2, 82.5)
- added C20: 47nF, Capacitor_SMD:C_0603_1608Metric, F.Cu at (142.4, 102.3)
- added C21: 0.1uF, Capacitor_SMD:C_0603_1608Metric, B.Cu at (101.2, 112.5)
- added C22: 10uF, Capacitor_SMD:C_0603_1608Metric, B.Cu at (103.0, 112.5)
- added C25: 0.1uF, Capacitor_SMD:C_0603_1608Metric, F.Cu at (149.6, 81.8)
- added C26: 0.1uF, Capacitor_SMD:C_0603_1608Metric, F.Cu at (160.2, 81.8)
- added C27: 0.1uF, Capacitor_SMD:C_0603_1608Metric, F.Cu at (119.6, 122.2)
- added C28: 0.1uF, Capacitor_SMD:C_0603_1608Metric, F.Cu at (130.4, 122.2)
- added C3: 33pF, Capacitor_SMD:C_0603_1608Metric, F.Cu at (144.2, 84.1)
- added C30: 0.1uF, Capacitor_SMD:C_0603_1608Metric, F.Cu at (95.4, 86.4)
- added C31: 10uF, Capacitor_SMD:C_0603_1608Metric, F.Cu at (103.2, 80.4)
- added C32: 1uF, Capacitor_SMD:C_0603_1608Metric, F.Cu at (104.9, 80.4)
- added C33: 0.1uF, Capacitor_SMD:C_0603_1608Metric, F.Cu at (106.6, 80.4)
- added C34: 10uF, Capacitor_SMD:C_0603_1608Metric, F.Cu at (95.4, 88.0)
- added C35: 10uF, Capacitor_SMD:C_0603_1608Metric, F.Cu at (84.3, 99.3)
- added C36: 10uF, Capacitor_SMD:C_0603_1608Metric, F.Cu at (87.5, 99.3)
- added C37: 10uF, Capacitor_SMD:C_0603_1608Metric, F.Cu at (99.7, 102.0)
- added C38: 10uF, Capacitor_SMD:C_0603_1608Metric, F.Cu at (91.0, 102.2)
- added C39: 10uF, Capacitor_SMD:C_0603_1608Metric, F.Cu at (150.4, 125.3)
- added C4: 1uF, Capacitor_SMD:C_0603_1608Metric, B.Cu at (143.6, 95.2)
- added C40: 0.1uF, Capacitor_SMD:C_0603_1608Metric, F.Cu at (148.7, 125.3)
- added C41: 0.1uF, Capacitor_SMD:C_0603_1608Metric, F.Cu at (143.1, 125.3)
- added C42: 10uF, Capacitor_SMD:C_0603_1608Metric, F.Cu at (141.4, 125.3)
- added C43: 0.1uF, Capacitor_SMD:C_0603_1608Metric, F.Cu at (148.7, 119.8)
- added C44: 10uF, Capacitor_SMD:C_0603_1608Metric, F.Cu at (150.4, 119.8)
- added C45: 0.1uF, Capacitor_SMD:C_0603_1608Metric, F.Cu at (143.1, 119.8)
- added C46: 10uF, Capacitor_SMD:C_0603_1608Metric, F.Cu at (141.4, 119.8)
- added C48: 10nF, Capacitor_SMD:C_0603_1608Metric, F.Cu at (143.6, 107.4)
- added C49: 10nF, Capacitor_SMD:C_0603_1608Metric, F.Cu at (143.6, 112.9)
- added C5: 10uF, Capacitor_SMD:C_0603_1608Metric, B.Cu at (146.4, 88.8)
- added C50: 0.1uF, Capacitor_SMD:C_0603_1608Metric, F.Cu at (163.4, 112.9)
- added C6: 0.1uF, Capacitor_SMD:C_0603_1608Metric, F.Cu at (150.0, 93.6)
- added C7: 0.1uF, Capacitor_SMD:C_0603_1608Metric, B.Cu at (144.7, 88.8)
- added C8: 0.1uF, Capacitor_SMD:C_0603_1608Metric, B.Cu at (142.2, 88.8)
- added C9: 10uF, Capacitor_SMD:C_0603_1608Metric, B.Cu at (146.0, 92.0)
- added D1: LED, LED_SMD:LED_0603_1608Metric, F.Cu at (84.4, 104.6)
- added D2: LED, LED_SMD:LED_0603_1608Metric, F.Cu at (84.4, 102.9)
- added FB1: 120E, Resistor_SMD:R_0603_1608Metric, F.Cu at (85.9, 99.3)
- added FB2: 120E, Resistor_SMD:R_0603_1608Metric, F.Cu at (139.7, 125.3)
- added J1: Conn_01x04_Pin, Connector_PinHeader_2.54mm:PinHeader_1x04_P2.54mm_Vertical, F.Cu at (94.1, 83.8)
- added J5: Conn_01x02_Pin, Connector_JST:JST_EH_B2B-EH-A_1x02_P2.50mm_Vertical, F.Cu at (108.8, 129.5)
- added R1: 100K, Resistor_SMD:R_0603_1608Metric, F.Cu at (152.5, 94.8)
- added R10: 100K, Resistor_SMD:R_0603_1608Metric, F.Cu at (135.1, 92.8)
- added R11: 100K, Resistor_SMD:R_0603_1608Metric, F.Cu at (132.2, 86.4)
- added R12: 100K, Resistor_SMD:R_0603_1608Metric, F.Cu at (132.2, 88.0)
- added R13: 100K, Resistor_SMD:R_0603_1608Metric, F.Cu at (135.1, 96.0)
- added R14: 0E, Resistor_SMD:R_0603_1608Metric, F.Cu at (153.3, 98.7)
- added R15: 0E, Resistor_SMD:R_0603_1608Metric, F.Cu at (153.3, 97.1)
- added R16: 20E, Resistor_SMD:R_0603_1608Metric, F.Cu at (144.0, 99.2)
- added R17: 20E, Resistor_SMD:R_0603_1608Metric, F.Cu at (140.8, 99.2)
- added R18: 10E, Resistor_SMD:R_0603_1608Metric, F.Cu at (142.4, 99.2)
- added R19: 0E, Resistor_SMD:R_0603_1608Metric, F.Cu at (159.4, 90.0)
- added R2: 100K, Resistor_SMD:R_0603_1608Metric, F.Cu at (121.2, 100.5)
- added R20: 0E, Resistor_SMD:R_0603_1608Metric, F.Cu at (159.4, 93.2)
- added R21: 10K, Resistor_SMD:R_0603_1608Metric, F.Cu at (101.2, 116.5)
- added R24: 10K, Resistor_SMD:R_0603_1608Metric, F.Cu at (149.6, 83.4)
- added R25: 10K, Resistor_SMD:R_0603_1608Metric, F.Cu at (160.2, 83.4)
- added R26: 10K, Resistor_SMD:R_0603_1608Metric, F.Cu at (119.6, 120.6)
- added R27: 10K, Resistor_SMD:R_0603_1608Metric, F.Cu at (130.4, 120.6)
- added R28: 10K, Resistor_SMD:R_0603_1608Metric, F.Cu at (99.5, 86.4)
- added R29: 0E, Resistor_SMD:R_0603_1608Metric, F.Cu at (105.6, 95.1)
- added R3: 1M, Resistor_SMD:R_0603_1608Metric, F.Cu at (141.9, 83.3)
- added R30: 0E, Resistor_SMD:R_0603_1608Metric, F.Cu at (105.6, 96.7)
- added R31: 5.1K, Resistor_SMD:R_0603_1608Metric, F.Cu at (92.2, 89.1)
- added R32: 5.1K, Resistor_SMD:R_0603_1608Metric, F.Cu at (92.1, 94.4)
- added R33: 2K, Resistor_SMD:R_0603_1608Metric, F.Cu at (89.1, 99.3)
- added R34: 1K, Resistor_SMD:R_0603_1608Metric, F.Cu at (91.0, 105.4)
- added R35: 1K, Resistor_SMD:R_0603_1608Metric, F.Cu at (91.0, 103.8)
- added R37: 0E, Resistor_SMD:R_0603_1608Metric, F.Cu at (157.8, 90.0)
- added R38: 10K, Resistor_SMD:R_0603_1608Metric, F.Cu at (142.0, 107.4)
- added R39: 10K, Resistor_SMD:R_0603_1608Metric, F.Cu at (142.0, 112.9)
- added R4: 100K, Resistor_SMD:R_0603_1608Metric, F.Cu at (128.9, 86.4)
- added R40: 10K, Resistor_SMD:R_0603_1608Metric, F.Cu at (165.2, 112.9)
- added R41: 10K, Resistor_SMD:R_0603_1608Metric, F.Cu at (102.6, 86.4)
- added R5: 100K, Resistor_SMD:R_0603_1608Metric, F.Cu at (153.3, 89.9)
- added R6: 100K, Resistor_SMD:R_0603_1608Metric, F.Cu at (153.3, 88.3)
- added R7: 100K, Resistor_SMD:R_0603_1608Metric, F.Cu at (153.3, 86.7)
- added R8: 100K, Resistor_SMD:R_0603_1608Metric, F.Cu at (153.3, 85.1)
- added R9: 100K, Resistor_SMD:R_0603_1608Metric, F.Cu at (135.1, 94.4)
- added SW3: SW_Push, Button_Switch_THT:SW_Tactile_SPST_Angled_PTS645Vx58-2LFS, F.Cu at (144.1, 76.5)
- added SW4: SW_Push, Button_Switch_THT:SW_Tactile_SPST_Angled_PTS645Vx58-2LFS, F.Cu at (154.7, 76.5)
- added SW5: SW_Push, Button_Switch_THT:SW_Tactile_SPST_Angled_PTS645Vx58-2LFS, F.Cu at (125.2, 127.5)
- added SW6: SW_Push, Button_Switch_THT:SW_Tactile_SPST_Angled_PTS645Vx58-2LFS, F.Cu at (135.9, 127.5)
- added SW8: SW_SPDT, Button_Switch_THT:SW_Slide_SPDT_Angled_CK_OS102011MA1Q, F.Cu at (143.9, 129.8)
- added SW9: RotaryEncoder_Switch, Rotary_Encoder:RotaryEncoder_Alps_EC11E-Switch_Vertical_H20mm, F.Cu at (146.2, 107.1)
- added U3: USBLC6-2SC6, Package_TO_SOT_SMD:SOT-23-6, F.Cu at (92.7, 91.8)
- added U5: XC6220B331MR, Package_TO_SOT_SMD:SOT-23-5, F.Cu at (145.9, 124.8)
- added U6: AP2112K-1.8, Package_TO_SOT_SMD:SOT-23-5, F.Cu at (145.9, 119.2)
- added Y1: AB308-12.288MHZ, GlobalFP:XTAL_AB308-12.288MHZ, F.Cu at (140.3, 83.3)
- J2, J3, J4, U1, U2, U4: moved to F.Cu
- moved H1 108.8 mm to (167.5, 127.2), turned to 90 degrees
- moved H3 83.7 mm to (167.5, 77.2), turned to 90 degrees
- moved J3 78.1 mm to (169.4, 90.8), turned to 180 degrees
- moved H2 70.8 mm to (87.5, 77.2), turned to 90 degrees
- moved H4 63.7 mm to (87.5, 127.2), turned to 90 degrees
- moved J2 46.3 mm to (91.4, 114.0), turned to -90 degrees
- moved J4 40.7 mm to (84.7, 91.8), turned to -90 degrees
- moved U1 29.3 mm to (142.4, 91.9)
- moved U4 20.7 mm to (94.4, 98.6), turned to 0 degrees
- moved U2 19.9 mm to (117.5, 85.3), turned to 0 degrees
Connections:
- J3 pad 1: GND -> /GBUFA
- J3 pad 2: /RIGHT_OUT -> /LEFTA
- J3 pad 3: /LEFT_OUT -> /RIGHTA
- U1 pad 37: GNDA -> GND
- U1 pad 40: GNDA -> GND
- U1 pad 41: GNDA -> GND
- U1 pad 47: GNDA -> GND
- U2 pad 12: unconnected-(U2-IO8-Pad12) -> /Rotary2
- U2 pad 13: Net-(U2-USB_D-) -> /DX-
- U2 pad 14: Net-(U2-USB_D+) -> /DX+
- U2 pad 15: unconnected-(U2-IO3-Pad15) -> /Rotary1
- U2 pad 17: unconnected-(U2-IO9-Pad17) -> /Card_Det
- U2 pad 23: unconnected-(U2-IO21-Pad23) -> /XDCS
- U2 pad 33: unconnected-(U2-IO40-Pad33) -> /Disp_SCL
- U2 pad 34: unconnected-(U2-IO41-Pad34) -> /Disp_SDA
- U2 pad 35: unconnected-(U2-IO42-Pad35) -> /XCS
- U2 pad 4: unconnected-(U2-IO4-Pad4) -> /R_S
- U2 pad 5: unconnected-(U2-IO5-Pad5) -> /Button1
- U2 pad 6: unconnected-(U2-IO6-Pad6) -> /Button2
- U2 pad 7: unconnected-(U2-IO7-Pad7) -> /Button3
- U2 pad 8: unconnected-(U2-IO15-Pad8) -> /Button4
- U2 pad 9: unconnected-(U2-IO16-Pad9) -> /DREQ
Routing:
- net +1V8: track 0.00 -> 87.5 mm, vias 0 -> 5
- net /VBAT_CHG: track 0.00 -> 87.4 mm, vias 0 -> 1
- net /R_S: track 0.00 -> 87.0 mm, vias 0 -> 1
- net /Button3: track 0.00 -> 77.8 mm, vias 0 -> 2
- net /DREQ: track 0.00 -> 73.2 mm, vias 0 -> 2
- net /Button4: track 0.00 -> 66.7 mm, vias 0 -> 2
- net /Rotary2: track 0.00 -> 66.4 mm, vias 0 -> 2
- net /MISO: track 0.00 -> 65.5 mm
- net /SCLK: track 0.00 -> 64.6 mm, vias 0 -> 3
- net /MOSI: track 0.00 -> 64.4 mm, vias 0 -> 3
- net /Button2: track 0.00 -> 61.3 mm, vias 0 -> 2
- net /VS_RST: track 0.00 -> 60.9 mm, vias 0 -> 4
- net VDDA: track 0.00 -> 54.2 mm, vias 0 -> 5
- net GND: track 0.00 -> 54.0 mm, vias 0 -> 51
- net /Button1: track 0.00 -> 51.1 mm, vias 0 -> 2
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- added copper zone on B.Cu, net +3V3
- added copper zone on F.Cu, net +3V3
- added copper zone on In1.Cu, net GND
- added copper zone on In2.Cu, net GND
- added copper zone on B.Cu, net VDDA
Other:
- board size 65 x 85 mm -> 90 x 60 mm
- board text added: "SynthWeave"

Commit message: Updated PCB routing
Parts:
- moved R12 1.00 mm to (133.2, 88.2)
- moved R11 0.98 mm to (133.2, 86.4)
- moved J4 0.28 mm to (85.0, 91.8)
- moved R10 0.20 mm to (135.1, 93.0)
- moved R13 0.20 mm to (135.1, 96.2)
- moved R9 0.20 mm to (135.1, 94.6)
Routing:
- net GND: track 54.0 -> 84.8 mm, vias 51 -> 74
- net +3V3: track 30.6 -> 33.3 mm, vias 23 -> 35
- net /D+: track 5.95 -> 4.82 mm
- net /RX: track 5.90 -> 4.84 mm
- net /VBUS: track 32.7 -> 31.7 mm
- net /GPIO5: track 6.35 -> 5.38 mm
- net /LEFTA: track 9.19 -> 8.49 mm
- net /D-: track 5.24 -> 5.80 mm
- net +1V8: track 87.5 -> 88.0 mm
Other:
- board text removed: "SynthWeave"
