File: PCB_Design/OpenWave_V1/OpenWave.kicad_sch (KiCad schematic)
At the start: 117 parts, among them J1 Conn_01x04_Pin, J2 Micro_SD_Card_Det1, J3 SJ1-3545N, J4 USB_C_Receptacle_USB2.0_16P, J5 Conn_01x02_Pin, SW1 SW_Push, SW2 SW_Push, SW3 SW_Push, SW4 SW_Push, SW5 SW_Push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

Commit message: Completed PCB Design, Updated Licences and Readme.
Parts:
- C47: footprint Capacitor_THT:C_Axial_L5.1mm_D3.1mm_P12.50mm_Horizontal -> Capacitor_THT:CP_Radial_D5.0mm_P2.00mm
- SW1, SW2: footprint Button_Switch_THT:SW_Tactile_SPST_Angled_PTS645Vx58-2LFS -> GlobalFP:TS3315A
Changed lines of the file:
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@@
 			)
 		)
-		(property "Footprint" "Button_Switch_THT:SW_Tactile_SPST_Angled_PTS645Vx58-2LFS"
+		(property "Footprint" "GlobalFP:TS3315A"
 			(at 349.25 26.67 0)
 			(effects
@@
 			)
 		)
-		(property "Footprint" "Capacitor_THT:C_Axial_L5.1mm_D3.1mm_P12.50mm_Horizontal"
+		(property "Footprint" "Capacitor_THT:CP_Radial_D5.0mm_P2.00mm"
 			(at 265.43 138.43 0)
 			(effects
@@
 			)
 		)
-		(property "Footprint" "Button_Switch_THT:SW_Tactile_SPST_Angled_PTS645Vx58-2LFS"
+		(property "Footprint" "GlobalFP:TS3315A"
 			(at 300.99 26.67 0)
 			(effects

Commit message: Added power indicators and silkscreen
Parts:
- added D3, D4: LED, LED_SMD:LED_0603_1608Metric, symbol Device:LED
- added R36, R42: 330E, Resistor_SMD:R_0603_1608Metric, symbol Device:R_Small
Connections:
- net +1V8: now also D4.2 (A)
- net +3V3: now also D3.2 (A)
- net GND: now also R36.1, R42.1
- new net: D3.1 (K), R36.2
- new net: D4.1 (K), R42.2

Commit message: Updated BOM,  Changed ESP pin defs.
Connections:
- net Rotary1: now also U2.25 (IO48); no longer U2.15 (IO3)
Changed lines of the file:
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@@
 	)
 	(no_connect
-		(at 62.23 91.44)
+		(at 31.75 58.42)
 	)
 	(no_connect
@@
 	(wire
 		(pts
+			(xy 62.23 91.44) (xy 82.55 91.44)
+		)
+		(stroke
+			(width 0)
+			(type default)
+		)
+	)
+	(wire
+		(pts
 			(xy 19.05 83.82) (xy 31.75 83.82)
 		)
@@
 	(wire
 		(pts
-			(xy 19.05 58.42) (xy 31.75 58.42)
-		)
-		(stroke
-			(width 0)
-			(type default)
-		)
-	)
-	(wire
-		(pts
 			(xy 262.89 36.83) (xy 265.43 36.83)
 		)
@@
 		)
 	)
+	(label "Rotary1"
+		(at 74.93 91.44 0)
+		(effects
+			(font
+				(size 1.27 1.27)
+			)
+			(justify left bottom)
+		)
+	)
 	(label "Button4"
 		(at 21.59 88.9 0)
@@
 		(effects
 			(font
-				(size 1.27 1.27)
-			)
-			(justify left bottom)
-		)
-	)
-	(label "Rotary1"
-		(at 21.59 58.42 0)
-		(effects
-			(font
